File: eagle/Galaksija keyboard matrix.sch (EAGLE design)
At the start: 58 parts

Commit message: New version Rev.2
Parts:
- removed JP1: to LS251, pinhead:PINHD-1X8
- removed JP2: to LS145, pinhead:PINHD-1X8
- added LED1: PWR, led:LED5MM
- added R1: 1k, rcl:R-EU_0207/10
- added S57: RST, switch-omron:40-XX
- added SV1: KBD, con-harting-ml:ML20
Connections:
- removed net IN0: JP1.8, S17.P, S17.P1, S25.P, S25.P1, S33.P, S33.P1, S41.P, S41.P1, S49.P, S49.P1, S9.P, S9.P1
- removed net IN1: JP1.7, S10.P, S10.P1, S18.P, S18.P1, S2.P, S2.P1, S26.P, S26.P1, S34.P, S34.P1, S42.P, S42.P1, S50.P, S50.P1
- removed net IN2: JP1.6, S11.P, S11.P1, S19.P, S19.P1, S27.P, S27.P1, S3.P, S3.P1, S35.P, S35.P1, S43.P, S43.P1, S51.P, S51.P1
- removed net IN3: JP1.5, S12.P, S12.P1, S20.P, S20.P1, S28.P, S28.P1, S36.P, S36.P1, S4.P, S4.P1, S44.P, S44.P1, S52.P, S52.P1
- removed net IN4: JP1.4, S13.P, S13.P1, S21.P, S21.P1, S29.P, S29.P1, S37.P, S37.P1, S45.P, S45.P1, S5.P, S5.P1, S53.P, S53.P1
- removed net IN5: JP1.3, S14.P, S14.P1, S22.P, S22.P1, S30.P, S30.P1, S38.P, S38.P1, S46.P, S46.P1, S54.P, S54.P1, S55.P, S55.P1, S6.P, S6.P1
- removed net IN6: JP1.2, S15.P, S15.P1, S23.P, S23.P1, S31.P, S31.P1, S39.P, S39.P1, S47.P, S47.P1, S7.P, S7.P1
- removed net IN7: JP1.1, S1.P, S1.P1, S16.P, S16.P1, S24.P, S24.P1, S32.P, S32.P1, S40.P, S40.P1, S48.P, S48.P1, S56.P, S56.P1, S8.P, S8.P1
- new net D7: S1.P, S1.P1, S16.P, S16.P1, S24.P, S24.P1, S32.P, S32.P1, S40.P, S40.P1, S48.P, S48.P1, S56.P, S56.P1, S8.P, S8.P1, SV1.4
- new net GND: LED1.C, SV1.2, SV1.20
- new net N$1: LED1.A, R1.2
- new net Q0: S2.S, S2.S1, S3.S, S3.S1, S4.S, S4.S1, S5.S, S5.S1, S6.S, S6.S1, S7.S, S7.S1, S8.S, S8.S1, SV1.3
- new net Q1: S10.S, S10.S1, S11.S, S11.S1, S12.S, S12.S1, S13.S, S13.S1, S14.S, S14.S1, S15.S, S15.S1, S16.S, S16.S1, S9.S, S9.S1, SV1.5
- new net Q2: S17.S, S17.S1, S18.S, S18.S1, S19.S, S19.S1, S20.S, S20.S1, S21.S, S21.S1, S22.S, S22.S1, S23.S, S23.S1, S24.S, S24.S1, SV1.7
- new net Q3: S1.S, S1.S1, S25.S, S25.S1, S26.S, S26.S1, S27.S, S27.S1, S28.S, S28.S1, S29.S, S29.S1, S30.S, S30.S1, S31.S, S31.S1, S32.S, S32.S1, S56.S, S56.S1, SV1.9
- new net Q4: S33.S, S33.S1, S34.S, S34.S1, S35.S, S35.S1, S36.S, S36.S1, S37.S, S37.S1, S38.S, S38.S1, S39.S, S39.S1, S40.S, S40.S1, SV1.11
- new net Q5: S41.S, S41.S1, S42.S, S42.S1, S43.S, S43.S1, S44.S, S44.S1, S45.S, S45.S1, S46.S, S46.S1, S47.S, S47.S1, S48.S, S48.S1, SV1.13
- new net Q6: S49.S, S49.S1, S50.S, S50.S1, S51.S, S51.S1, S52.S, S52.S1, S53.S, S53.S1, S54.S, S54.S1, S55.S, S55.S1, SV1.15
- new net RST: S57.S, S57.S1, SV1.19
- new net VCC: R1.1, S57.P, S57.P1, SV1.1
- net D0: now also S17.P, S17.P1, S25.P, S25.P1, S33.P, S33.P1, S41.P, S41.P1, S49.P, S49.P1, S9.P, S9.P1, SV1.18; no longer JP2.1, S2.S, S2.S1, S3.S, S3.S1, S4.S, S4.S1, S5.S, S5.S1, S6.S, S6.S1, S7.S, S7.S1, S8.S, S8.S1
- net D1: now also S10.P, S10.P1, S18.P, S18.P1, S2.P, S2.P1, S26.P, S26.P1, S34.P, S34.P1, S42.P, S42.P1, S50.P, S50.P1, SV1.16; no longer JP2.2, S10.S, S10.S1, S11.S, S11.S1, S12.S, S12.S1, S13.S, S13.S1, S14.S, S14.S1, S15.S, S15.S1, S16.S, S16.S1, S9.S, S9.S1
- net D2: now also S11.P, S11.P1, S19.P, S19.P1, S27.P, S27.P1, S3.P, S3.P1, S35.P, S35.P1, S43.P, S43.P1, S51.P, S51.P1, SV1.14; no longer JP2.3, S17.S, S17.S1, S18.S, S18.S1, S19.S, S19.S1, S20.S, S20.S1, S21.S, S21.S1, S22.S, S22.S1, S23.S, S23.S1, S24.S, S24.S1
- net D3: now also S12.P, S12.P1, S20.P, S20.P1, S28.P, S28.P1, S36.P, S36.P1, S4.P, S4.P1, S44.P, S44.P1, S52.P, S52.P1, SV1.12; no longer JP2.4, S1.S, S1.S1, S25.S, S25.S1, S26.S, S26.S1, S27.S, S27.S1, S28.S, S28.S1, S29.S, S29.S1, S30.S, S30.S1, S31.S, S31.S1, S32.S, S32.S1, S56.S, S56.S1
- net D4: now also S13.P, S13.P1, S21.P, S21.P1, S29.P, S29.P1, S37.P, S37.P1, S45.P, S45.P1, S5.P, S5.P1, S53.P, S53.P1, SV1.10; no longer JP2.5, S33.S, S33.S1, S34.S, S34.S1, S35.S, S35.S1, S36.S, S36.S1, S37.S, S37.S1, S38.S, S38.S1, S39.S, S39.S1, S40.S, S40.S1
- net D5: now also S14.P, S14.P1, S22.P, S22.P1, S30.P, S30.P1, S38.P, S38.P1, S46.P, S46.P1, S54.P, S54.P1, S55.P, S55.P1, S6.P, S6.P1, SV1.8; no longer JP2.6, S41.S, S41.S1, S42.S, S42.S1, S43.S, S43.S1, S44.S, S44.S1, S45.S, S45.S1, S46.S, S46.S1, S47.S, S47.S1, S48.S, S48.S1
- net D6: now also S15.P, S15.P1, S23.P, S23.P1, S31.P, S31.P1, S39.P, S39.P1, S47.P, S47.P1, S7.P, S7.P1, SV1.6; no longer JP2.7, S49.S, S49.S1, S50.S, S50.S1, S51.S, S51.S1, S52.S, S52.S1, S53.S, S53.S1, S54.S, S54.S1, S55.S, S55.S1
Other:
- note added: "Rev.2"
- note removed: "Rev. 1"
