File: eagle/Galaksija keyboard adapter.brd (EAGLE design)
At the start: 60.9 x 38.2 mm, 4 parts

Commit message: finished keyboard revision 3
Parts:
- moved JP2 1.27 mm to (52.1, 24.1)
- moved JP5 1.27 mm to (52.1, 7.62)
- moved JP1 1.27 mm to (16.5, 24.1)
Routing:
- net RST: track 79.4 -> 72.0 mm
- net GND: track 73.8 -> 78.3 mm
- net VCC: track 43.2 -> 44.5 mm
- net Q1: track 45.3 -> 46.6 mm
- net Q0: track 45.3 -> 46.6 mm
- net D5: track 12.3 -> 13.5 mm
- net D4: track 12.3 -> 13.5 mm
- net Q2: track 45.3 -> 46.6 mm
- net D2: track 12.6 -> 13.5 mm
- net Q4: track 45.8 -> 46.6 mm
- net Q6: track 45.8 -> 46.6 mm
- net D6: track 12.8 -> 13.5 mm
- net D3: track 12.8 -> 13.5 mm
- net D1: track 12.8 -> 13.5 mm
- net Q3: track 46.0 -> 46.6 mm
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Other:
- board size 60.9 x 38.2 mm -> 55.9 x 38.2 mm
- board text added: "Adapter 2"
- board text removed: "KBD"
