File: eagle/rev2/Galaksija keyboard matrix.sch (EAGLE design)
At the start: 63 parts

Commit message: Rev3 narrower version with modified ENTER key
Parts:
- removed S58, S59: Return, switch-omron:40-XX
- removed S60: RST2, switch-omron:10-XX
Connections:
- net D0: no longer S58.P, S58.P1, S59.P, S59.P1
- net Q6: no longer S58.S, S58.S1, S59.S, S59.S1
- net RST: no longer S60.S, S60.S1
- net VCC: no longer S60.P, S60.P1
Changed lines of the file:
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@@
 <part name="LED1" library="led" library_urn="urn:adsk.eagle:library:259" deviceset="LED" device="5MM" package3d_urn="urn:adsk.eagle:package:15799/2" value="PWR"/>
 <part name="R1" library="rcl" library_urn="urn:adsk.eagle:library:334" deviceset="R-EU_" device="0207/10" package3d_urn="urn:adsk.eagle:package:23491/2" value="1k"/>
-<part name="S58" library="switch-omron" library_urn="urn:adsk.eagle:library:377" deviceset="40-XX" device="" package3d_urn="urn:adsk.eagle:package:27483/1" value="Return"/>
-<part name="S59" library="switch-omron" library_urn="urn:adsk.eagle:library:377" deviceset="40-XX" device="" package3d_urn="urn:adsk.eagle:package:27483/1" value="Return"/>
-<part name="S60" library="switch-omron" library_urn="urn:adsk.eagle:library:377" deviceset="10-XX" device="" package3d_urn="urn:adsk.eagle:package:27496/1" value="RST2"/>
 </parts>
 <sheets>
@@
 </instance>
 <instance part="S57" gate="1" x="-5.08" y="109.22" smashed="yes" rot="R270">
-<attribute name="NAME" x="3.556" y="105.918" size="1.778" layer="95"/>
-<attribute name="VALUE" x="3.683" y="107.95" size="1.778" layer="96"/>
+<attribute name="NAME" x="-12.7" y="113.03" size="1.778" layer="95"/>
+<attribute name="VALUE" x="-1.905" y="113.03" size="1.778" layer="96"/>
 </instance>
 <instance part="LED1" gate="G$1" x="-68.58" y="83.82" smashed="yes">
@@
 <attribute name="NAME" x="-67.0814" y="97.79" size="1.778" layer="95" rot="R270"/>
 <attribute name="VALUE" x="-71.882" y="97.79" size="1.778" layer="96" rot="R270"/>
-</instance>
-<instance part="S58" gate="1" x="139.7" y="83.82" smashed="yes" rot="R270">
-<attribute name="NAME" x="132.08" y="87.63" size="1.778" layer="95"/>
-<attribute name="VALUE" x="142.875" y="87.63" size="1.778" layer="96"/>
-</instance>
-<instance part="S59" gate="1" x="139.7" y="99.06" smashed="yes" rot="R270">
-<attribute name="NAME" x="132.08" y="102.87" size="1.778" layer="95"/>
-<attribute name="VALUE" x="142.875" y="102.87" size="1.778" layer="96"/>
-</instance>
-<instance part="S60" gate="1" x="-5.08" y="104.14" smashed="yes" rot="R270">
-<attribute name="NAME" x="3.81" y="101.092" size="1.778" layer="95"/>
-<attribute name="VALUE" x="3.683" y="103.378" size="1.778" layer="96"/>
 </instance>
 </instances>
@@
 <wire x1="144.78" y1="-5.08" x2="147.32" y2="-5.08" width="0.1524" layer="91"/>
 <pinref part="SV1" gate="1" pin="15"/>
-<wire x1="147.32" y1="73.66" x2="147.32" y2="81.28" width="0.1524" layer="91"/>
-<wire x1="147.32" y1="81.28" x2="147.32" y2="83.82" width="0.1524" layer="91"/>
-<wire x1="147.32" y1="83.82" x2="147.32" y2="93.98" width="0.1524" layer="91"/>
+<wire x1="147.32" y1="73.66" x2="147.32" y2="93.98" width="0.1524" layer="91"/>
 <wire x1="147.32" y1="93.98" x2="-22.86" y2="93.98" width="0.1524" layer="91"/>
 <junction x="147.32" y="73.66"/>
 <label x="148.082" y="92.456" size="1.778" layer="95"/>
-<pinref part="S58" gate="1" pin="S1"/>
-<wire x1="144.78" y1="81.28" x2="147.32" y2="81.28" width="0.1524" layer="91"/>
-<junction x="147.32" y="81.28"/>
-<pinref part="S58" gate="1" pin="S"/>
-<wire x1="144.78" y1="83.82" x2="147.32" y2="83.82" width="0.1524" layer="91"/>
-<junction x="147.32" y="83.82"/>
-<pinref part="S59" gate="1" pin="S1"/>
-<wire x1="144.78" y1="96.52" x2="147.32" y2="96.52" width="0.1524" layer="91"/>
-<wire x1="147.32" y1="96.52" x2="147.32" y2="93.98" width="0.1524" layer="91"/>
-<junction x="147.32" y="93.98"/>
-<pinref part="S59" gate="1" pin="S"/>
-<wire x1="144.78" y1="99.06" x2="147.32" y2="99.06" width="0.1524" layer="91"/>
-<wire x1="147.32" y1="99.06" x2="147.32" y2="96.52" width="0.1524" layer="91"/>
-<junction x="147.32" y="96.52"/>
 </segment>
 </net>
@@
 <pinref part="SV1" gate="1" pin="18"/>
 <wire x1="-60.96" y1="96.52" x2="-38.1" y2="96.52" width="0.1524" layer="91"/>
-<pinref part="S58" gate="1" pin="P"/>
-<wire x1="132.08" y1="73.66" x2="132.08" y2="81.28" width="0.1524" layer="91"/>
-<wire x1="132.08" y1="81.28" x2="132.08" y2="83.82" width="0.1524" layer="91"/>
-<wire x1="132.08" y1="83.82" x2="134.62" y2="83.82" width="0.1524" layer="91"/>
-<junction x="132.08" y="73.66"/>
-<pinref part="S58" gate="1" pin="P1"/>
-<wire x1="134.62" y1="81.28" x2="132.08" y2="81.28" width="0.1524" layer="91"/>
-<junction x="132.08" y="81.28"/>
-<pinref part="S59" gate="1" pin="P"/>
-<wire x1="134.62" y1="99.06" x2="132.08" y2="99.06" width="0.1524" layer="91"/>
-<wire x1="132.08" y1="99.06" x2="132.08" y2="96.52" width="0.1524" layer="91"/>
-<junction x="132.08" y="83.82"/>
-<pinref part="S59" gate="1" pin="P1"/>
-<wire x1="132.08" y1="96.52" x2="132.08" y2="83.82" width="0.1524" layer="91"/>
-<wire x1="134.62" y1="96.52" x2="132.08" y2="96.52" width="0.1524" layer="91"/>
-<junction x="132.08" y="96.52"/>
 </segment>
 </net>
@@
 <pinref part="SV1" gate="1" pin="1"/>
 <wire x1="-22.86" y1="76.2" x2="-17.78" y2="76.2" width="0.1524" layer="91"/>
-<wire x1="-17.78" y1="76.2" x2="-17.78" y2="101.6" width="0.1524" layer="91"/>
+<wire x1="-17.78" y1="76.2" x2="-17.78" y2="106.68" width="0.1524" layer="91"/>
 <pinref part="R1" gate="G$1" pin="1"/>
-<wire x1="-17.78" y1="101.6" x2="-17.78" y2="104.14" width="0.1524" layer="91"/>
-<wire x1="-17.78" y1="104.14" x2="-17.78" y2="106.68" width="0.1524" layer="91"/>
 <wire x1="-17.78" y1="106.68" x2="-17.78" y2="109.22" width="0.1524" layer="91"/>
 <wire x1="-17.78" y1="109.22" x2="-68.58" y2="109.22" width="0.1524" layer="91"/>
@@
 <wire x1="-10.16" y1="106.68" x2="-17.78" y2="106.68" width="0.1524" layer="91"/>
 <junction x="-17.78" y="106.68"/>
-<pinref part="S60" gate="1" pin="P1"/>
-<wire x1="-10.16" y1="101.6" x2="-17.78" y2="101.6" width="0.1524" layer="91"/>
-<junction x="-17.78" y="101.6"/>
-<pinref part="S60" gate="1" pin="P"/>
-<wire x1="-10.16" y1="104.14" x2="-17.78" y2="104.14" width="0.1524" layer="91"/>
-<junction x="-17.78" y="104.14"/>
 </segment>
 </net>
@@
 <pinref part="SV1" gate="1" pin="19"/>
 <wire x1="-22.86" y1="99.06" x2="2.54" y2="99.06" width="0.1524" layer="91"/>
-<wire x1="2.54" y1="99.06" x2="2.54" y2="101.6" width="0.1524" layer="91"/>
+<wire x1="2.54" y1="99.06" x2="2.54" y2="106.68" width="0.1524" layer="91"/>
 <pinref part="S57" gate="1" pin="S"/>
-<wire x1="2.54" y1="101.6" x2="2.54" y2="104.14" width="0.1524" layer="91"/>
-<wire x1="2.54" y1="104.14" x2="2.54" y2="106.68" width="0.1524" layer="91"/>
 <wire x1="2.54" y1="106.68" x2="2.54" y2="109.22" width="0.1524" layer="91"/>
 <wire x1="2.54" y1="109.22" x2="0" y2="109.22" width="0.1524" layer="91"/>
@@
 <wire x1="0" y1="106.68" x2="2.54" y2="106.68" width="0.1524" layer="91"/>
 <junction x="2.54" y="106.68"/>
-<pinref part="S60" gate="1" pin="S"/>
-<wire x1="0" y1="104.14" x2="2.54" y2="104.14" width="0.1524" layer="91"/>
-<junction x="2.54" y="104.14"/>
-<pinref part="S60" gate="1" pin="S1"/>
-<wire x1="0" y1="101.6" x2="2.54" y2="101.6" width="0.1524" layer="91"/>
-<junction x="2.54" y="101.6"/>
-</segment>
-</net>
+</segment>
+</net>
